File: mouseDesign.kicad_pcb (KiCad board)
At the start: 2 copper layers, 31 parts, among them J1 USB_C_Receptacle, J2 JST_CONN, Q2 AO8810, U1 MCP1700T-2502E-MB, U3 USBLC6-2SC6, U4 DW01A, U5 MAX17048

Commit message: Added MCU
Parts:
- added U6: nRF52840, Package_DFN_QFN:Nordic_AQFN-73-1EP_7x7mm_P0.5mm, F.Cu at (96.5, 66.0)

Commit message: Update PCB layout and project settings, ignore KiCad autosave and logs
Parts:
- added R5: 4.7k, PCM_SparkFun-Resistor:R_0603_1608Metric, F.Cu at (104.8, 66.5)
- moved F2 8.66 mm to (123.0, 59.4)
- moved U6 8.61 mm to (101.8, 59.2)
- moved J1 3.39 mm to (125.0, 54.3), turned to 180 degrees
Connections:
- U3 pad 4: Net-(TP2-Pad1) -> /DATA_N
- U3 pad 6: Net-(TP1-Pad1) -> /DATA_P
- U6 pad A18: unconnected-(U6-DEC2-PadA18) -> Net-(C4-+)
- U6 pad A22: Net-(U6-VDD-PadA22) -> /3V3
- U6 pad AC5: unconnected-(U6-DECUSB-PadAC5) -> Net-(C13--)
- U6 pad AD14: Net-(U6-VDD-PadA22) -> /3V3
- U6 pad AD2: unconnected-(U6-VBUS-PadAD2) -> /VUSB
- U6 pad AD23: Net-(U6-VDD-PadA22) -> /3V3
- U6 pad AD4: unconnected-(U6-D--PadAD4) -> /DATA_N
- U6 pad AD6: unconnected-(U6-D+-PadAD6) -> /DATA_P
- U6 pad B1: Net-(U6-VDD-PadA22) -> /3V3
- U6 pad B5: unconnected-(U6-DEC4-PadB5) -> Net-(C7-+)
- U6 pad B7: Net-(U6-VSS-PadB7) -> GND
- U6 pad C1: unconnected-(U6-DEC1-PadC1) -> Net-(C10-+)
- U6 pad D23: unconnected-(U6-DEC3-PadD23) -> Net-(C6-+)
- U6 pad E24: unconnected-(U6-DEC6-PadE24) -> Net-(C9-+)
- U6 pad EP: Net-(U6-VSS-PadB7) -> GND
- U6 pad F23: unconnected-(U6-VSS_PA-PadF23) -> GND1-RF
- U6 pad N24: unconnected-(U6-DEC5-PadN24) -> Net-(C8-+)
- U6 pad W1: Net-(U6-VDD-PadA22) -> /3V3
- U6 pad Y2: unconnected-(U6-VDDH-PadY2) -> /3V3
